File: Eletronics/BLE_POV_clock_v2.0/BLE_POV_clock_v2.0.brd (EAGLE design)
At the start: 150 x 15 mm, 148 parts, among them P0.28 PUSHBUTTON_2X4X3.5

Commit message: BLE_POV_clock_v2.0 final version
Parts:
- removed MICRO_USB: USBSMALLGND, 0000_GV_connectors:MICROUSB_SMALLGND
- added BAT+, GND_1: PAD_50X100MIL, 0000_GV_connectors:PAD_50X100MIL
- added CC1_PDN, CC2_PDN: (no value), 0000_GV_resistors:0603-RES
- added U$11: CR2032CHINA, 0000_GV_batteries:CR2032_CHINA_HOLDER
- added U$19: USB-C_6PIN, 0000_GV_connectors:USCX-06FX-XXMX-01
- added U$20: CR2032-SMD, 0000_GV_batteries:CR2032
- moved REG 21.4 mm to (26.0, 7.51), turned to 0 degrees
- moved HPUP 16.1 mm to (28.7, 10.1)
- moved R_PWR_L 15.6 mm to (16.5, 14.0)
- moved HALL 14.3 mm to (20.3, 13.4), turned to 0 degrees
- moved PWR_L 14.0 mm to (14.0, 14.0), turned to 0 degrees
- moved IR_SENSOR 13.9 mm to (21.2, 8.49), turned to 180 degrees
- moved BAT1 13.0 mm to (18.2, 3.00), turned to 260 degrees
- moved BAT 12.1 mm to (136.0, 2.50)
- moved P0.28 11.0 mm to (26.3, 14.0)
- moved IPUP2 10.8 mm to (40.8, 12.2), turned to 270 degrees
- moved IPUP 10.8 mm to (39.4, 12.2), turned to 270 degrees
- moved MPU6050 10.6 mm to (33.2, 11.8)
- moved IR_R 9.78 mm to (17.0, 12.1), turned to 270 degrees
- moved 2477 8.65 mm to (120.0, 7.50), turned to 156 degrees
- moved C_VIN 8.28 mm to (103.4, 13.7)
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Connections:
- new net N$4: CC2_PDN.2, U$19.CC2
- new net N$9: CC1_PDN.2, U$19.CC1
- net BAT: now also GND_1.P$1, U$11.+1, U$11.+2, U$20.V+5, U$20.V+6
- net GND: now also BAT+.P$1, CC1_PDN.1, CC2_PDN.1, U$11.-, U$19.GND1, U$19.GND2, U$19.SHIELD1, U$19.SHIELD2, U$19.SHIELD3, U$19.SHIELD4, U$20.GND; no longer MICRO_USB.5, MICRO_USB.5.GND1, MICRO_USB.5.GND4
- net USB_VIN: now also U$19.VBUS1, U$19.VBUS2; no longer MICRO_USB.1
Routing:
- net 3V3: track 166.9 -> 129.0 mm, vias 8 -> 5
- net VIN_SW: track 35.1 -> 12.2 mm
- net GND: track 338.1 -> 320.4 mm, vias 12 -> 11
- net BAT: track 198.2 -> 186.0 mm, vias 2 -> 4
- net SCL: track 30.9 -> 20.3 mm
- net SDA: track 30.5 -> 20.0 mm
- net SENSOR: track 61.5 -> 52.1 mm, vias 3 -> 2
- net RED2: track 144.5 -> 136.1 mm, vias 1 -> 5
- net N$9: track 0.00 -> 7.59 mm
- net FET_M: track 22.4 -> 17.1 mm
- net USB_VIN: track 86.9 -> 91.3 mm
- net N$4: track 0.00 -> 3.22 mm
- net BLUE_S1: track 30.9 -> 27.8 mm
- net GREEN_S1: track 26.5 -> 23.4 mm
- net N$12: track 4.83 -> 7.15 mm
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Other:
- board size 150 x 15 mm -> 133 x 15 mm
