File: Eletronics/BLE_POV_clock_v2.0/BLE_POV_clock_v2.0.sch (EAGLE design)
At the start: 147 parts, among them P0.28 PUSHBUTTON_2X4X3.5

Commit message: BLE_POV_clock_v2.0 final version
Parts:
- removed MICRO_USB: USBSMALLGND, 0000_GV_connectors:USBSMALLGND
- added BAT+, GND_1: PAD_50X100MIL, 0000_GV_connectors:PAD_50X100MIL
- added CC1_PDN, CC2_PDN: (no value), 0000_GV_resistors:RESISTOR0603-RES
- added U$11: CR2032CHINA, 0000_GV_batteries:CR2032CHINA
- added U$19: USB-C_6PIN, 0000_GV_connectors:USB-C_6PIN
- added U$20: CR2032-SMD, 0000_GV_batteries:CR2032-SMD
Connections:
- new net N$4: CC2_PDN.2, U$19.CC2
- new net N$9: CC1_PDN.2, U$19.CC1
- net BAT: now also GND_1.P$1, U$11.+, U$20.+
- net GND: now also BAT+.P$1, CC1_PDN.1, CC2_PDN.1, U$11.-, U$19.GND, U$20.-; no longer MICRO_USB.5.GND
- net USB_VIN: now also U$19.VBUS; no longer MICRO_USB.1.VCC
Other:
- moved on the sheet: BAT, BAT1, PWR_L, R_PWR_L
